File: mainboard.sch (EAGLE design)
At the start: 28 parts, among them J1 AVR_SPI_PRG_6PTH, U1 ATMEGA328P, U2 3.3V, U3 5V, U4 MMA7660FCR1

Commit message: Added rtc
Parts:
- added IC1: DS1307, dallas-1:DS1307
- added Q1: 32.768 kHz, adafruit:CRYSTALTC38H
- added U$2: (no value), adafruit:CR1220SMT
Connections:
- new net N$7: IC1.VBAT, U$2.+
- new net N$8: IC1.X1, Q1.2
- new net N$9: IC1.X2, Q1.1
- net +5V: now also IC1.VCC
- net GND: now also IC1.GND, U$2.-
- net SCL: now also IC1.SCL
- net SDA: now also IC1.SDA
Other:
- note added: "RTC"
Changed lines of the file:
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@@
 <layer number="54" name="bGND_GNDA" color="1" fill="9" visible="no" active="no"/>
 <layer number="56" name="wert" color="7" fill="1" visible="no" active="no"/>
+<layer number="57" name="tCAD" color="7" fill="1" visible="no" active="no"/>
 <layer number="91" name="Nets" color="2" fill="1" visible="yes" active="yes"/>
 <layer number="92" name="Busses" color="1" fill="1" visible="yes" active="yes"/>
@@
 <layer number="108" name="tplace-old" color="10" fill="1" visible="yes" active="yes"/>
 <layer number="109" name="ref-old" color="11" fill="1" visible="yes" active="yes"/>
+<layer number="110" name="fp0" color="7" fill="1" visible="no" active="yes"/>
+<layer number="111" name="LPC17xx" color="7" fill="1" visible="yes" active="yes"/>
+<layer number="112" name="tSilk" color="7" fill="1" visible="yes" active="yes"/>
 <layer number="116" name="Patch_BOT" color="9" fill="4" visible="yes" active="yes"/>
 <layer number="121" name="_tsilk" color="7" fill="1" visible="yes" active="yes"/>
 <layer number="122" name="_bsilk" color="7" fill="1" visible="yes" active="yes"/>
+<layer number="123" name="tTestmark" color="7" fill="1" visible="no" active="yes"/>
+<layer number="124" name="bTestmark" color="7" fill="1" visible="no" active="yes"/>
 <layer number="125" name="_tNames" color="7" fill="1" visible="yes" active="yes"/>
+<layer number="126" name="_bNames" color="7" fill="1" visible="yes" active="yes"/>
+<layer number="127" name="_tValues" color="7" fill="1" visible="yes" active="yes"/>
+<layer number="128" name="_bValues" color="7" fill="1" visible="yes" active="yes"/>
+<layer number="131" name="tAdjust" color="7" fill="1" visible="no" active="yes"/>
+<layer number="132" name="bAdjust" color="7" fill="1" visible="no" active="yes"/>
 <layer number="144" name="Drill_legend" color="7" fill="1" visible="yes" active="yes"/>
+<layer number="150" name="Notes" color="7" fill="1" visible="no" active="yes"/>
 <layer number="151" name="HeatSink" color="7" fill="1" visible="yes" active="yes"/>
+<layer number="152" name="_bDocu" color="7" fill="1" visible="yes" active="yes"/>
+<layer number="153" name="FabDoc1" color="6" fill="1" visible="no" active="no"/>
+<layer number="154" name="FabDoc2" color="2" fill="1" visible="no" active="no"/>
+<layer number="155" name="FabDoc3" color="7" fill="15" visible="no" active="no"/>
 <layer number="199" name="Contour" color="7" fill="1" visible="yes" active="yes"/>
 <layer number="200" name="200bmp" color="1" fill="10" visible="yes" active="yes"/>
@@
 <layer number="223" name="223bmp" color="24" fill="1" visible="no" active="no"/>
 <layer number="224" name="224bmp" color="25" fill="1" visible="no" active="no"/>
+<layer number="248" name="Housing" color="7" fill="1" visible="yes" active="yes"/>
+<layer number="249" name="Edge" color="7" fill="1" visible="yes" active="yes"/>
 <layer number="250" name="Descript" color="3" fill="1" visible="no" active="no"/>
 <layer number="251" name="SMDround" color="12" fill="11" visible="no" active="no"/>
@@
 <part name="GND18" library="supply1" deviceset="GND" device=""/>
 <part name="R11" library="SparkFun-Resistors" deviceset="RESISTOR" device="0603-RES" value="1.8K"/>
+<part name="IC1" library="dallas-1" deviceset="DS1307" device=""/>
+<part name="GND19" library="supply1" deviceset="GND" device=""/>
+<part name="U$2" library="adafruit" deviceset="CR1220" device="SMT"/>
+<part name="GND20" library="supply1" deviceset="GND" device=""/>
+<part name="Q1" library="adafruit" deviceset="CRYSTAL" device="TC38H" value="32.768 kHz"/>
 </parts>
 <sheets>
@@
 <text x="73.66" y="106.68" size="1.778" layer="91">REGULATORS</text>
 <text x="175.26" y="109.22" size="1.778" layer="91">I2C pullups</text>
+<text x="243.84" y="-15.24" size="1.778" layer="91">RTC</text>
 </plain>
 <instances>
@@
 <instance part="GND18" gate="1" x="124.46" y="86.36"/>
 <instance part="R11" gate="G$1" x="198.12" y="93.98" rot="R90"/>
+<instance part="IC1" gate="G$1" x="243.84" y="-38.1"/>
+<instance part="GND19" gate="1" x="228.6" y="-45.72" rot="R270"/>
+<instance part="U$2" gate="G$1" x="218.44" y="-60.96"/>
+<instance part="GND20" gate="1" x="213.36" y="-63.5"/>
+<instance part="Q1" gate="G$1" x="220.98" y="-33.02" rot="R90"/>
 </instances>
 <busses>
@@
 <pinref part="GND18" gate="1" pin="GND"/>
 </segment>
+<segment>
+<pinref part="IC1" gate="G$1" pin="GND"/>
+<pinref part="GND19" gate="1" pin="GND"/>
+</segment>
+<segment>
+<pinref part="U$2" gate="G$1" pin="-"/>
+<pinref part="GND20" gate="1" pin="GND"/>
+</segment>
 </net>
 <net name="+5V" class="0">
@@
 <label x="66.04" y="99.06" size="1.778" layer="95"/>
 </segment>
+<segment>
+<pinref part="IC1" gate="G$1" pin="VCC"/>
+<wire x1="254" y1="-30.48" x2="266.7" y2="-30.48" width="0.1524" layer="91"/>
+<label x="266.7" y="-30.48" size="1.778" layer="95"/>
+</segment>
 </net>
 <net name="N$4" class="0">
@@
 <label x="190.5" y="-33.02" size="1.778" layer="95"/>
 </segment>
+<segment>
+<pinref part="IC1" gate="G$1" pin="SDA"/>
+<wire x1="254" y1="-45.72" x2="266.7" y2="-45.72" width="0.1524" layer="91"/>
+<label x="266.7" y="-45.72" size="1.778" layer="95"/>
+</segment>
 </net>
 <net name="SCL" class="0">
@@
 <wire x1="142.24" y1="-40.64" x2="132.08" y2="-40.64" width="0.1524" layer="91"/>
 <label x="132.08" y="-40.64" size="1.778" layer="95"/>
+</segment>
+<segment>
+<pinref part="IC1" gate="G$1" pin="SCL"/>
+<wire x1="254" y1="-40.64" x2="266.7" y2="-40.64" width="0.1524" layer="91"/>
+<label x="266.7" y="-40.64" size="1.778" layer="95"/>
 </segment>
 </net>
@@
 </segment>
 </net>
+<net name="N$7" class="0">
+<segment>
+<pinref part="U$2" gate="G$1" pin="+"/>
+<wire x1="223.52" y1="-58.42" x2="223.52" y2="-40.64" width="0.1524" layer="91"/>
+<pinref part="IC1" gate="G$1" pin="VBAT"/>
+<wire x1="223.52" y1="-40.64" x2="231.14" y2="-40.64" width="0.1524" layer="91"/>
+</segment>
+</net>
+<net name="N$8" class="0">
+<segment>
+<pinref part="Q1" gate="G$1" pin="2"/>
+<pinref part="IC1" gate="G$1" pin="X1"/>
+<wire x1="220.98" y1="-30.48" x2="231.14" y2="-30.48" width="0.1524" layer="91"/>
+</segment>
+</net>
+<net name="N$9" class="0">
+<segment>
+<pinref part="Q1" gate="G$1" pin="1"/>
+<pinref part="IC1" gate="G$1" pin="X2"/>
+<wire x1="220.98" y1="-35.56" x2="231.14" y2="-35.56" width="0.1524" layer="91"/>
+</segment>
+</net>

Commit message: Add switching regulator to board
Parts:
- added D1: MBRS320, diode:SCHOTTKY-DIODESMC
- added IC2: LM2596S, national-semiconductor:LM2596S
- added J2: (no value), SparkFun-Connectors:JST_2MM_MALE
- added L1: 33uH, srr1280:L-SRR1280
Connections:
- new net BAT+: IC2.VIN, J2.+
- new net N$10: D1.C, IC2.OUT, L1.1
- net GND: now also D1.A, IC2.!ON!/OFF, IC2.GND, J2.-
Other:
- note added: "+6V Buck converter"
Changed lines of the file:
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@@
 <part name="GND20" library="supply1" deviceset="GND" device=""/>
 <part name="Q1" library="adafruit" deviceset="CRYSTAL" device="TC38H" value="32.768 kHz"/>
+<part name="IC2" library="national-semiconductor" deviceset="LM2596" device="S"/>
+<part name="GND21" library="supply1" deviceset="GND" device=""/>
+<part name="J2" library="SparkFun-Connectors" deviceset="JST_2MM_MALE" device=""/>
+<part name="GND22" library="supply1" deviceset="GND" device=""/>
+<part name="GND23" library="supply1" deviceset="GND" device=""/>
+<part name="D1" library="diode" deviceset="SCHOTTKY-DIODE" device="SMC" value="MBRS320"/>
+<part name="L1" library="srr1280" deviceset="L" device="-SRR1280" value="33uH"/>
 </parts>
 <sheets>
@@
 <text x="175.26" y="109.22" size="1.778" layer="91">I2C pullups</text>
 <text x="243.84" y="-15.24" size="1.778" layer="91">RTC</text>
+<text x="248.92" y="109.22" size="1.778" layer="91">+6V Buck converter</text>
 </plain>
 <instances>
@@
 <instance part="GND20" gate="1" x="213.36" y="-63.5"/>
 <instance part="Q1" gate="G$1" x="220.98" y="-33.02" rot="R90"/>
+<instance part="IC2" gate="G$1" x="264.16" y="88.9"/>
+<instance part="GND21" gate="1" x="233.68" y="81.28"/>
+<instance part="J2" gate="G$1" x="238.76" y="48.26" rot="R90"/>
+<instance part="GND22" gate="1" x="254" y="45.72"/>
+<instance part="GND23" gate="1" x="294.64" y="83.82"/>
+<instance part="D1" gate="G$1" x="294.64" y="88.9" rot="R90"/>
+<instance part="L1" gate="G$1" x="309.88" y="91.44" rot="R90"/>
 </instances>
 <busses>
@@
 <pinref part="GND20" gate="1" pin="GND"/>
 </segment>
+<segment>
+<pinref part="IC2" gate="G$1" pin="GND"/>
+<pinref part="GND21" gate="1" pin="GND"/>
+<wire x1="233.68" y1="83.82" x2="243.84" y2="83.82" width="0.1524" layer="91"/>
+<pinref part="IC2" gate="G$1" pin="!ON!/OFF"/>
+<wire x1="243.84" y1="83.82" x2="251.46" y2="83.82" width="0.1524" layer="91"/>
+<wire x1="251.46" y1="88.9" x2="243.84" y2="88.9" width="0.1524" layer="91"/>
+<wire x1="243.84" y1="88.9" x2="243.84" y2="83.82" width="0.1524" layer="91"/>
+<junction x="243.84" y="83.82"/>
+</segment>
+<segment>
+<pinref part="J2" gate="G$1" pin="-"/>
+<pinref part="GND22" gate="1" pin="GND"/>
+<wire x1="254" y1="48.26" x2="243.84" y2="48.26" width="0.1524" layer="91"/>
+</segment>
+<segment>
+<pinref part="GND23" gate="1" pin="GND"/>
+<pinref part="D1" gate="G$1" pin="A"/>
+</segment>
 </net>
 <net name="+5V" class="0">
@@
 </segment>
 </net>
+<net name="BAT+" class="0">
+<segment>
+<pinref part="IC2" gate="G$1" pin="VIN"/>
+<wire x1="251.46" y1="93.98" x2="233.68" y2="93.98" width="0.1524" layer="91"/>
+<wire x1="233.68" y1="93.98" x2="233.68" y2="101.6" width="0.1524" layer="91"/>
+<label x="233.68" y="101.6" size="1.778" layer="95"/>
+</segment>
+<segment>
+<pinref part="J2" gate="G$1" pin="+"/>
+<wire x1="243.84" y1="50.8" x2="254" y2="50.8" width="0.1524" layer="91"/>
+<label x="254" y="50.8" size="1.778" layer="95"/>
+</segment>
+</net>
+<net name="N$10" class="0">
+<segment>
+<pinref part="IC2" gate="G$1" pin="OUT"/>
+<pinref part="D1" gate="G$1" pin="C"/>
+<wire x1="276.86" y1="91.44" x2="302.26" y2="91.44" width="0.1524" layer="91"/>
+<pinref part="L1" gate="G$1" pin="1"/>
+<junction x="302.26" y="91.44"/>
+<wire x1="302.26" y1="91.44" x2="294.64" y2="91.44" width="0.1524" layer="91"/>
+</segment>
+</net>

Commit message: Finish 6V buck converter, add battery voltage sense
Parts:
- removed POWER: (no value), con-ptr500:AK500/2
- added C5: 330 uF, SparkFun-Capacitors:CAP_POLE
- added C6: 470uF, SparkFun-Capacitors:CAP_POLG
- added C7: 0.1uF, SparkFun-Capacitors:CAP0603-CAP
- added R12: 240, SparkFun-Resistors:RESISTOR0603
- added R13: 931, SparkFun-Resistors:RESISTOR0603
- added R14: 1M, SparkFun-Resistors:RESISTOR0603
- added R15: 780k, SparkFun-Resistors:RESISTOR0603
Connections:
- new net A1: U1.PC1(ADC1)
- new net A2: U1.PC2(ADC2)
- new net BAT_SENSE: C7.1, R14.1, R15.2, U1.PC0(ADC0)
- new net D4: U1.PD4(XCK/T0)
- new net D7: U1.PD7(AIN1)
- new net N$11: IC2.FB, R12.2, R13.1
- net +6V: now also C5.+, L1.2, R13.2; no longer POWER-1.KL
- net BAT+: now also C6.+, R14.2
- net GND: now also C5.-, C6.-, C7.2, R12.1, R15.1; no longer POWER-2.KL
Other:
- note added: "BAT conn and sensor"
Changed lines of the file:
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@@
 </classes>
 <parts>
-<part name="POWER" library="con-ptr500" deviceset="AK500/2" device=""/>
 <part name="U1" library="SparkFun-DigitalIC" deviceset="ATMEGA328_SMT" device="" value="ATMEGA328P"/>
-<part name="GND1" library="supply1" deviceset="GND" device=""/>
 <part name="GND2" library="supply1" deviceset="GND" device=""/>
 <part name="C1" library="SparkFun-Capacitors" deviceset="CAP" device="0603-CAP" value="0.1uF"/>
@@
 <part name="D1" library="diode" deviceset="SCHOTTKY-DIODE" device="SMC" value="MBRS320"/>
 <part name="L1" library="srr1280" deviceset="L" device="-SRR1280" value="33uH"/>
+<part name="C5" library="SparkFun-Capacitors" deviceset="CAP_POL" device="E" value="330 uF"/>
+<part name="GND1" library="supply1" deviceset="GND" device=""/>
+<part name="R12" library="SparkFun-Resistors" deviceset="RESISTOR" device="0603" value="240"/>
+<part name="GND24" library="supply1" deviceset="GND" device=""/>
+<part name="R13" library="SparkFun-Resistors" deviceset="RESISTOR" device="0603" value="931"/>
+<part name="C6" library="SparkFun-Capacitors" deviceset="CAP_POL" device="G" value="470uF"/>
+<part name="R14" library="SparkFun-Resistors" deviceset="RESISTOR" device="0603" value="1M"/>
+<part name="R15" library="SparkFun-Resistors" deviceset="RESISTOR" device="0603" value="780k"/>
+<part name="C7" library="SparkFun-Capacitors" deviceset="CAP" device="0603-CAP" value="0.1uF"/>
+<part name="GND25" library="supply1" deviceset="GND" device=""/>
+<part name="GND26" library="supply1" deviceset="GND" device=""/>
 </parts>
 <sheets>
@@
 <text x="243.84" y="-15.24" size="1.778" layer="91">RTC</text>
 <text x="248.92" y="109.22" size="1.778" layer="91">+6V Buck converter</text>
+<text x="241.3" y="58.42" size="1.778" layer="91">BAT conn and sensor</text>
 </plain>
 <instances>
-<instance part="POWER" gate="-1" x="2.54" y="96.52"/>
-<instance part="POWER" gate="-2" x="2.54" y="91.44"/>
 <instance part="U1" gate="G$1" x="88.9" y="33.02"/>
-<instance part="GND1" gate="1" x="7.62" y="88.9"/>
 <instance part="GND2" gate="1" x="43.18" y="91.44" rot="R270"/>
 <instance part="C1" gate="G$1" x="71.12" y="91.44"/>
@@
 <instance part="D1" gate="G$1" x="294.64" y="88.9" rot="R90"/>
 <instance part="L1" gate="G$1" x="309.88" y="91.44" rot="R90"/>
+<instance part="C5" gate="G$1" x="322.58" y="88.9"/>
+<instance part="GND1" gate="1" x="322.58" y="81.28"/>
+<instance part="R12" gate="G$1" x="279.4" y="104.14"/>
+<instance part="GND24" gate="1" x="271.78" y="104.14" rot="R270"/>
+<instance part="R13" gate="G$1" x="289.56" y="104.14"/>
+<instance part="C6" gate="G$1" x="238.76" y="88.9"/>
+<instance part="R14" gate="G$1" x="241.3" y="22.86" rot="R90"/>
+<instance part="R15" gate="G$1" x="241.3" y="10.16" rot="R90"/>
+<instance part="C7" gate="G$1" x="251.46" y="7.62"/>
+<instance part="GND25" gate="1" x="241.3" y="2.54"/>
+<instance part="GND26" gate="1" x="251.46" y="2.54"/>
 </instances>
 <busses>
@@
 <nets>
 <net name="+6V" class="0">
-<segment>
-<pinref part="POWER" gate="-1" pin="KL"/>
-<wire x1="7.62" y1="96.52" x2="12.7" y2="96.52" width="0.1524" layer="91"/>
-<label x="10.16" y="99.06" size="1.778" layer="95"/>
-</segment>
 <segment>
 <wire x1="45.72" y1="96.52" x2="40.64" y2="96.52" width="0.1524" layer="91"/>
@@
 <junction x="91.44" y="96.52"/>
 </segment>
+<segment>
+<pinref part="L1" gate="G$1" pin="2"/>
+<pinref part="C5" gate="G$1" pin="+"/>
+<wire x1="322.58" y1="91.44" x2="317.5" y2="91.44" width="0.1524" layer="91"/>
+<wire x1="322.58" y1="91.44" x2="335.28" y2="91.44" width="0.1524" layer="91"/>
+<junction x="322.58" y="91.44"/>
+<label x="332.74" y="91.44" size="1.778" layer="95"/>
+<pinref part="R13" gate="G$1" pin="2"/>
+<wire x1="294.64" y1="104.14" x2="322.58" y2="104.14" width="0.1524" layer="91"/>
+<wire x1="322.58" y1="104.14" x2="322.58" y2="91.44" width="0.1524" layer="91"/>
+</segment>
 </net>
 <net name="GND" class="0">
-<segment>
-<pinref part="POWER" gate="-2" pin="KL"/>
-<pinref part="GND1" gate="1" pin="GND"/>
-</segment>
 <segment>
 <pinref part="C1" gate="G$1" pin="2"/>
@@
 <pinref part="IC2" gate="G$1" pin="GND"/>
 <pinref part="GND21" gate="1" pin="GND"/>
-<wire x1="233.68" y1="83.82" x2="243.84" y2="83.82" width="0.1524" layer="91"/>
+<wire x1="233.68" y1="83.82" x2="238.76" y2="83.82" width="0.1524" layer="91"/>
 <pinref part="IC2" gate="G$1" pin="!ON!/OFF"/>
+<wire x1="238.76" y1="83.82" x2="243.84" y2="83.82" width="0.1524" layer="91"/>
 <wire x1="243.84" y1="83.82" x2="251.46" y2="83.82" width="0.1524" layer="91"/>
 <wire x1="251.46" y1="88.9" x2="243.84" y2="88.9" width="0.1524" layer="91"/>
 <wire x1="243.84" y1="88.9" x2="243.84" y2="83.82" width="0.1524" layer="91"/>
 <junction x="243.84" y="83.82"/>
+<pinref part="C6" gate="G$1" pin="-"/>
+<junction x="238.76" y="83.82"/>
 </segment>
 <segment>
@@
 <pinref part="GND23" gate="1" pin="GND"/>
 <pinref part="D1" gate="G$1" pin="A"/>
+</segment>
+<segment>
+<pinref part="C5" gate="G$1" pin="-"/>
+<pinref part="GND1" gate="1" pin="GND"/>
+</segment>
+<segment>
+<pinref part="R12" gate="G$1" pin="1"/>
+<pinref part="GND24" gate="1" pin="GND"/>
+</segment>
+<segment>
+<pinref part="R15" gate="G$1" pin="1"/>
+<pinref part="GND25" gate="1" pin="GND"/>
+</segment>
+<segment>
+<pinref part="C7" gate="G$1" pin="2"/>
+<pinref part="GND26" gate="1" pin="GND"/>
 </segment>
 </net>
@@
 <net name="BAT+" class="0">
 <segment>
-<pinref part="IC2" gate="G$1" pin="VIN"/>
-<wire x1="251.46" y1="93.98" x2="233.68" y2="93.98" width="0.1524" layer="91"/>
 <wire x1="233.68" y1="93.98" x2="233.68" y2="101.6" width="0.1524" layer="91"/>
 <label x="233.68" y="101.6" size="1.778" layer="95"/>
+<pinref part="IC2" gate="G$1" pin="VIN"/>
+<wire x1="233.68" y1="93.98" x2="238.76" y2="93.98" width="0.1524" layer="91"/>
+<pinref part="C6" gate="G$1" pin="+"/>
+<wire x1="238.76" y1="93.98" x2="251.46" y2="93.98" width="0.1524" layer="91"/>
+<wire x1="238.76" y1="91.44" x2="238.76" y2="93.98" width="0.1524" layer="91"/>
+<junction x="238.76" y="93.98"/>
 </segment>
 <segment>
@@
 <wire x1="243.84" y1="50.8" x2="254" y2="50.8" width="0.1524" layer="91"/>
 <label x="254" y="50.8" size="1.778" layer="95"/>
+</segment>
+<segment>
+<wire x1="241.3" y1="35.56" x2="241.3" y2="27.94" width="0.1524" layer="91"/>
+<label x="241.3" y="35.56" size="1.778" layer="95"/>
+<pinref part="R14" gate="G$1" pin="2"/>
 </segment>
 </net>
@@
 </segment>
 </net>
+<net name="N$11" class="0">
+<segment>
+<pinref part="IC2" gate="G$1" pin="FB"/>
+<wire x1="276.86" y1="86.36" x2="284.48" y2="86.36" width="0.1524" layer="91"/>
+<wire x1="284.48" y1="86.36" x2="284.48" y2="104.14" width="0.1524" layer="91"/>
+<pinref part="R12" gate="G$1" pin="2"/>
+<pinref part="R13" gate="G$1" pin="1"/>
+<junction x="284.48" y="104.14"/>
+</segment>
+</net>
+<net name="BAT_SENSE" class="0">
+<segment>
+<pinref part="U1" gate="G$1" pin="PC0(ADC0)"/>
+<wire x1="114.3" y1="58.42" x2="121.92" y2="58.42" width="0.1524" layer="91"/>
+<label x="119.38" y="58.42" size="1.778" layer="95"/>
+</segment>
+<segment>
+<pinref part="R14" gate="G$1" pin="1"/>
+<pinref part="R15" gate="G$1" pin="2"/>
+<wire x1="241.3" y1="17.78" x2="241.3" y2="15.24" width="0.1524" layer="91"/>
+<pinref part="C7" gate="G$1" pin="1"/>
+<wire x1="241.3" y1="17.78" x2="251.46" y2="17.78" width="0.1524" layer="91"/>
+<wire x1="251.46" y1="17.78" x2="251.46" y2="12.7" width="0.1524" layer="91"/>
+<wire x1="251.46" y1="17.78" x2="266.7" y2="17.78" width="0.1524" layer="91"/>
+<junction x="251.46" y="17.78"/>
+<label x="264.16" y="17.78" size="1.778" layer="95"/>
+</segment>
+</net>
+<net name="A1" class="0">
+<segment>
+<pinref part="U1" gate="G$1" pin="PC1(ADC1)"/>
+<wire x1="114.3" y1="55.88" x2="121.92" y2="55.88" width="0.1524" layer="91"/>
+<label x="124.46" y="55.88" size="1.778" layer="95"/>
+</segment>
+</net>
+<net name="A2" class="0">
+<segment>
+<pinref part="U1" gate="G$1" pin="PC2(ADC2)"/>
+<wire x1="114.3" y1="53.34" x2="121.92" y2="53.34" width="0.1524" layer="91"/>
+<label x="124.46" y="53.34" size="1.778" layer="95"/>
+</segment>
+</net>
+<net name="D4" class="0">
+<segment>
+<pinref part="U1" gate="G$1" pin="PD4(XCK/T0)"/>
+<wire x1="114.3" y1="25.4" x2="121.92" y2="25.4" width="0.1524" layer="91"/>
+<label x="124.46" y="25.4" size="1.778" layer="95"/>
+</segment>
+</net>
+<net name="D7" class="0">
+<segment>
+<pinref part="U1" gate="G$1" pin="PD7(AIN1)"/>
+<wire x1="114.3" y1="17.78" x2="121.92" y2="17.78" width="0.1524" layer="91"/>
+<label x="124.46" y="17.78" size="1.778" layer="95"/>
+</segment>
+</net>

Commit message: Initial crack at board design
Parts:
- added JP12: Extra, SparkFun-Connectors:M06SIP
Connections:
- net +5V: now also JP12.2
- net A1: now also JP12.6
- net A2: now also JP12.5
- net D4: now also JP12.4
- net D7: now also JP12.3
- net GND: now also JP12.1
Other:
- note added: "Extra connections"
Changed lines of the file:
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@@
 <part name="GND25" library="supply1" deviceset="GND" device=""/>
 <part name="GND26" library="supply1" deviceset="GND" device=""/>
+<part name="GND27" library="supply1" deviceset="GND" device=""/>
+<part name="JP12" library="SparkFun-Connectors" deviceset="M06" device="SIP" value="Extra"/>
 </parts>
 <sheets>
@@
 <text x="248.92" y="109.22" size="1.778" layer="91">+6V Buck converter</text>
 <text x="241.3" y="58.42" size="1.778" layer="91">BAT conn and sensor</text>
+<text x="289.56" y="-7.62" size="1.778" layer="91">Extra connections</text>
 </plain>
 <instances>
@@
 <instance part="GND25" gate="1" x="241.3" y="2.54"/>
 <instance part="GND26" gate="1" x="251.46" y="2.54"/>
+<instance part="GND27" gate="1" x="314.96" y="-35.56" rot="R90"/>
+<instance part="JP12" gate="G$1" x="297.18" y="-30.48"/>
 </instances>
 <busses>
@@
 <pinref part="GND26" gate="1" pin="GND"/>
 </segment>
+<segment>
+<pinref part="JP12" gate="G$1" pin="1"/>
+<pinref part="GND27" gate="1" pin="GND"/>
+<wire x1="312.42" y1="-35.56" x2="302.26" y2="-35.56" width="0.1524" layer="91"/>
+</segment>
 </net>
 <net name="+5V" class="0">
@@
 <wire x1="254" y1="-30.48" x2="266.7" y2="-30.48" width="0.1524" layer="91"/>
 <label x="266.7" y="-30.48" size="1.778" layer="95"/>
+</segment>
+<segment>
+<pinref part="JP12" gate="G$1" pin="2"/>
+<wire x1="302.26" y1="-33.02" x2="312.42" y2="-33.02" width="0.1524" layer="91"/>
+<label x="314.96" y="-33.02" size="1.778" layer="95"/>
 </segment>
 </net>
@@
 <junction x="251.46" y="17.78"/>
 <label x="264.16" y="17.78" size="1.778" layer="95"/>
+<junction x="241.3" y="17.78"/>
 </segment>
 </net>
@@
 <label x="124.46" y="55.88" size="1.778" layer="95"/>
 </segment>
+<segment>
+<pinref part="JP12" gate="G$1" pin="6"/>
+<wire x1="302.26" y1="-22.86" x2="312.42" y2="-22.86" width="0.1524" layer="91"/>
+<label x="314.96" y="-22.86" size="1.778" layer="95"/>
+</segment>
 </net>
 <net name="A2" class="0">
@@
 <label x="124.46" y="53.34" size="1.778" layer="95"/>
 </segment>
+<segment>
+<pinref part="JP12" gate="G$1" pin="5"/>
+<wire x1="302.26" y1="-25.4" x2="312.42" y2="-25.4" width="0.1524" layer="91"/>
+<label x="314.96" y="-25.4" size="1.778" layer="95"/>
+</segment>
 </net>
 <net name="D4" class="0">
@@
 <label x="124.46" y="25.4" size="1.778" layer="95"/>
 </segment>
+<segment>
+<pinref part="JP12" gate="G$1" pin="4"/>
+<wire x1="302.26" y1="-27.94" x2="312.42" y2="-27.94" width="0.1524" layer="91"/>
+<label x="314.96" y="-27.94" size="1.778" layer="95"/>
+</segment>
 </net>
 <net name="D7" class="0">
@@
 <label x="124.46" y="17.78" size="1.778" layer="95"/>
 </segment>
+<segment>
+<pinref part="JP12" gate="G$1" pin="3"/>
+<wire x1="302.26" y1="-30.48" x2="312.42" y2="-30.48" width="0.1524" layer="91"/>
+<label x="314.96" y="-30.48" size="1.778" layer="95"/>
+</segment>
 </net>
 </nets>
 </sheet>
 </sheets>
+<errors>
+</errors>
 </schematic>
 </drawing>
